Commit message: added onshape exported urdf

File: ros2/src/camera_mount_description/urdf/camera_mount.urdf.xacro (robot description, xacro)
@@ -1,70 +1,182 @@
 <?xml version="1.0"?>
-<robot name="camera_mount" xmlns:xacro="http://www.ros.org/wiki/xacro">
-  <!-- PLACEHOLDER GEOMETRY: boxes and approximate offsets standing in for the
-       OnShape design, which hasn't been exported yet. Joint names ("yaw", "pitch")
-       and joint limits are real, matching
-       ros2/src/camera_mount_bridge/config/servos.json (that copy, not python's;
-       see project notes on why the two are kept separate). If you recalibrate,
-       update the limit values below too.
-       Standalone for now: camera_mount_base_link is not yet attached to anything.
-       Attaching to the G1 head is a static joint once its parent link and offset
-       are known; everything below is unaffected by that. -->
-  <material name="mount_grey">
-    <color rgba="0.6 0.6 0.6 1.0"/>
-  </material>
-  <material name="camera_black">
-    <color rgba="0.1 0.1 0.1 1.0"/>
-  </material>
-  <link name="camera_mount_base_link"/>
-  <link name="yaw_link">
-    <visual>
-      <geometry>
-        <box size="0.03 0.03 0.03"/>
-      </geometry>
-      <material name="mount_grey"/>
-    </visual>
-  </link>
-  <joint name="yaw" type="revolute">
-    <parent link="camera_mount_base_link"/>
-    <child link="yaw_link"/>
-    <origin xyz="0 0 0" rpy="0 0 0"/>
-    <axis xyz="0 0 1"/>
-    <limit lower="-1.5374" upper="1.5727" effort="1.0" velocity="1.0"/>
-  </joint>
-  <link name="pitch_link">
-    <visual>
-      <geometry>
-        <box size="0.03 0.03 0.03"/>
-      </geometry>
-      <material name="mount_grey"/>
-    </visual>
-  </link>
-  <joint name="pitch" type="revolute">
-    <parent link="yaw_link"/>
-    <child link="pitch_link"/>
-    <origin xyz="0 0 0.03" rpy="0 0 0"/>
-    <axis xyz="0 1 0"/>
-    <limit lower="-1.3548" upper="0.9237" effort="1.0" velocity="1.0"/>
-  </joint>
-  <link name="camera_link">
-    <visual>
-      <geometry>
-        <box size="0.02 0.04 0.02"/>
-      </geometry>
-      <material name="camera_black"/>
-    </visual>
-  </link>
-  <joint name="camera_mount_joint" type="fixed">
-    <parent link="pitch_link"/>
-    <child link="camera_link"/>
-    <origin xyz="0.03 0 0" rpy="0 0 0"/>
-  </joint>
-  <!-- REP-103 optical-frame convention (Z-forward, X-right, Y-down) for anything
-       downstream that expects it (camera_info, image_proc, vision pipelines). -->
-  <link name="camera_optical_frame"/>
-  <joint name="camera_optical_joint" type="fixed">
-    <parent link="camera_link"/>
-    <child link="camera_optical_frame"/>
-    <origin xyz="0 0 0" rpy="-1.5707963 0 -1.5707963"/>
-  </joint>
+<!-- Hand-maintained: onshape_export/onshape.urdf is regenerated by onshape-to-robot
+     and overwritten on the next OnShape export, so it is not edited in place. This
+     file wraps its camera_mount_base_link/camera_mount_yaw_link/camera_mount_pitch_link
+     links and yaw/pitch joints, minus the raw "Part d455" visual/collision (replaced
+     below by the real sensor_d455 macro, which adds camera_link plus the actual
+     depth/color/infra/imu TF frames the RealSense driver publishes against, unlike
+     onshape.urdf's plain mesh which had none of those). If the links change in a
+     fresh OnShape export, re-sync them here by hand; the sensor_d455 origin below
+     (measured against onshape.urdf's "Part d455" mesh placement, which is unaffected
+     by link renames) would also need recomputing if the camera's position in the
+     design changes; see this package's README for the full re-sync walkthrough.
+     Packaged as a xacro:macro (not a standalone <robot>) so it can be attached
+     anywhere: standalone for bench testing (see camera_mount_standalone.urdf.xacro)
+     or, later, into the G1's own URDF via
+       <xacro:include filename="$(find camera_mount_description)/urdf/camera_mount.urdf.xacro"/>
+       <xacro:camera_mount parent="<g1_head_link>">
+         <origin xyz="..." rpy="..."/>
+       </xacro:camera_mount>
+     once the mounting link and offset on the real head are known. -->
+<robot xmlns:xacro="http://www.ros.org/wiki/xacro">
+  <xacro:include filename="$(find realsense2_description)/urdf/_d455.urdf.xacro"/>
+  <xacro:macro name="camera_mount" params="parent *origin">
+    <joint name="camera_mount_joint" type="fixed">
+      <parent link="${parent}"/>
+      <child link="camera_mount_base_link"/>
+      <xacro:insert_block name="origin"/>
+    </joint>
+    <!-- Link camera_mount_base_link -->
+    <link name="camera_mount_base_link">
+      <inertial>
+        <origin xyz="0.0186709 -5.01832e-07 0.532413" rpy="0 0 0"/>
+        <mass value="0.0125893"/>
+        <inertia ixx="2.85959e-06" ixy="2.39e-10" ixz="7.3616e-07" iyy="1.08803e-05" iyz="-1.5e-11" izz="1.35768e-05"/>
+      </inertial>
+      <!-- Part camera_mount_base_link -->
+      <visual>
+        <origin xyz="0 0 0" rpy="0 -0 0"/>
+        <geometry>
+          <mesh filename="package://camera_mount_description/urdf/assets/camera_mount_base_link.stl"/>
+        </geometry>
+        <material name="camera_mount_base_link_material">
+          <color rgba="0.647059 0.647059 0.647059 1"/>
+        </material>
+      </visual>
+      <collision>
+        <origin xyz="0 0 0" rpy="0 -0 0"/>
+        <geometry>
+          <mesh filename="package://camera_mount_description/urdf/assets/camera_mount_base_link.stl"/>
+        </geometry>
+      </collision>
+      <!-- Part dc15_a01_case_f_dummy -->
+      <visual>
+        <origin xyz="0.056648 0 0.550718" rpy="0 0 -1.5708"/>
+        <geometry>
+          <mesh filename="package://camera_mount_description/urdf/assets/dc15_a01_case_f_dummy.stl"/>
+        </geometry>
+        <material name="dc15_a01_case_f_dummy_material">
+          <color rgba="0.917647 0.917647 0.917647 1"/>
+        </material>
+      </visual>
+      <collision>
+        <origin xyz="0.056648 0 0.550718" rpy="0 0 -1.5708"/>
+        <geometry>
+          <mesh filename="package://camera_mount_description/urdf/assets/dc15_a01_case_f_dummy.stl"/>
+        </geometry>
+      </collision>
+      <!-- Part base_mount -->
+      <visual>
+        <origin xyz="0 0 0" rpy="0 -0 -0"/>
+        <geometry>
+          <mesh filename="package://camera_mount_description/urdf/assets/base_mount.stl"/>
+        </geometry>
+        <material name="base_mount_material">
+          <color rgba="0.972549 0.529412 0.00392157 1"/>
+        </material>
+      </visual>
+      <collision>
+        <origin xyz="0 0 0" rpy="0 -0 -0"/>
+        <geometry>
+          <mesh filename="package://camera_mount_description/urdf/assets/base_mount.stl"/>
+        </geometry>
+      </collision>
+    </link>
+    <!-- Link camera_mount_yaw_link -->
+    <link name="camera_mount_yaw_link">
+      <inertial>
+        <origin xyz="-4.64212e-06 0.00142735 -0.00376553" rpy="0 0 0"/>
+        <mass value="0.00610061"/>
+        <inertia ixx="6.93909e-07" ixy="-5.31e-10" ixz="-1.38e-10" iyy="8.57171e-07" iyz="4.2567e-08" izz="1.21949e-06"/>
+      </inertial>
+      <!-- Part dc15_a01_case_f_dummy_2 -->
+      <visual>
+        <origin xyz="-0.00794467 -0.0170259 -0.013" rpy="3.13834 1.5708 0"/>
+        <geometry>
+          <mesh filename="package://camera_mount_description/urdf/assets/dc15_a01_case_f_dummy.stl"/>
+        </geometry>
+        <material name="dc15_a01_case_f_dummy_2_material">
+          <color rgba="0.917647 0.917647 0.917647 1"/>
+        </material>
+      </visual>
+      <collision>
+        <origin xyz="-0.00794467 -0.0170259 -0.013" rpy="3.13834 1.5708 0"/>
+        <geometry>
+          <mesh filename="package://camera_mount_description/urdf/assets/dc15_a01_case_f_dummy.stl"/>
+        </geometry>
+      </collision>
+      <!-- Part camera_mount_yaw_link -->
+      <visual>
+        <origin xyz="0 0 0" rpy="-3.14159 0 0.00325227"/>
+        <geometry>
+          <mesh filename="package://camera_mount_description/urdf/assets/camera_mount_yaw_link.stl"/>
+        </geometry>
+        <material name="camera_mount_yaw_link_material">
+          <color rgba="0.615686 0.811765 0.929412 1"/>
+        </material>
+      </visual>
+      <collision>
+        <origin xyz="0 0 0" rpy="-3.14159 0 0.00325227"/>
+        <geometry>
+          <mesh filename="package://camera_mount_description/urdf/assets/camera_mount_yaw_link.stl"/>
+        </geometry>
+      </collision>
+    </link>
+    <!-- Link camera_mount_pitch_link -->
+    <link name="camera_mount_pitch_link">
+      <inertial>
+        <origin xyz="0.0153805 -0 0.0124131" rpy="0 0 0"/>
+        <mass value="0.013697"/>
+        <inertia ixx="1.29622e-05" ixy="0" ixz="-3.20967e-07" iyy="1.28138e-05" iyz="-0" izz="8.57555e-07"/>
+      </inertial>
+      <!-- Part camera_mount_pitch_link (the "Part d455" visual/collision that
+           onshape.urdf has here is intentionally dropped: sensor_d455 below supplies
+           the real mesh, correctly tied to camera_link instead of floating
+           disconnected from TF) -->
+      <visual>
+        <origin xyz="0.0189975 -0 0.0145" rpy="-1.5708 -1.5708 0"/>
+        <geometry>
+          <mesh filename="package://camera_mount_description/urdf/assets/camera_mount_pitch_link.stl"/>
+        </geometry>
+        <material name="camera_mount_pitch_link_material">
+          <color rgba="0.615686 0.811765 0.929412 1"/>
+        </material>
+      </visual>
+      <collision>
+        <origin xyz="0.0189975 -0 0.0145" rpy="-1.5708 -1.5708 0"/>
+        <geometry>
+          <mesh filename="package://camera_mount_description/urdf/assets/camera_mount_pitch_link.stl"/>
+        </geometry>
+      </collision>
+    </link>
+    <!-- Joint from camera_mount_yaw_link to camera_mount_pitch_link -->
+    <joint name="pitch" type="revolute">
+      <origin xyz="-0.0144446 -0.0170471 -0.013" rpy="-1.5708 0.0247295 -1.56754"/>
+      <parent link="camera_mount_yaw_link"/>
+      <child link="camera_mount_pitch_link"/>
+      <axis xyz="0 0 1"/>
+      <limit effort="10" velocity="10" lower="-3.141592653589793" upper="3.141592653589793"/>
+    </joint>
+    <!-- Joint from camera_mount_base_link to camera_mount_yaw_link -->
+    <joint name="yaw" type="revolute">
+      <origin xyz="0.056648 0 0.557218" rpy="-3.14159 0 -1.5708"/>
+      <parent link="camera_mount_base_link"/>
+      <child link="camera_mount_yaw_link"/>
+      <axis xyz="0 0 1"/>
+      <limit effort="10" velocity="10" lower="-3.141592653589793" upper="3.141592653589793"/>
+    </joint>
+    <!-- D455: origin solved from onshape.urdf's "Part d455" mesh placement composed
+         against realsense2_description's own bottom_screw_frame->mesh offsets. The
+         camera is rear-screw-mounted in this design, not bottom-mounted, but that
+         only changes which physical screws hold it: bottom_screw_frame is just a
+         fixed reference point on the rigid D455 body, unaffected by which holes are
+         actually used. Verified: recomposing this origin against sensor_d455's
+         internal offsets reproduces onshape.urdf's original mesh placement exactly
+         (both d455 meshes, ours and realsense2_description's, share the same local
+         origin convention, confirmed by comparing STL bounding boxes: identical
+         124x26x29mm dimensions, matching center offsets to sub-mm noise). -->
+    <xacro:sensor_d455 parent="camera_mount_pitch_link" name="camera" use_nominal_extrinsics="true">
+      <origin xyz="0.029198 -0.0145 0.0145" rpy="-1.570796 0 0"/>
+    </xacro:sensor_d455>
+  </xacro:macro>
 </robot>
