Commit message: update the urdf

File: ros2/src/camera_mount_description/onshape_export/onshape.urdf (robot description, URDF)
Before this commit: robot camera_mount, 3 links, 2 joints
Links:
- added link base_link, mass 1e-9
Joints:
- added joint base_link_frame: type fixed, parent camera_mount_base_link, child base_link, origin xyz=0 0 0 rpy=0 -0 -0, axis 0 0 0
- joint yaw: origin xyz=0.056648 0 0.557218 rpy=-3.14159 0 -1.5708 -> xyz=0.0574997 0 0.022 rpy=-3.14159 0 -1.5708

File: ros2/src/camera_mount_description/urdf/camera_mount.urdf.xacro (robot description, xacro)
@@ -30,5 +30,5 @@
     <link name="camera_mount_base_link">
       <inertial>
-        <origin xyz="0.0186709 -5.01832e-07 0.532413" rpy="0 0 0"/>
+        <origin xyz="0.0195225 -5.01832e-07 -0.00280466" rpy="0 0 0"/>
         <mass value="0.0125893"/>
         <inertia ixx="2.85959e-06" ixy="2.39e-10" ixz="7.3616e-07" iyy="1.08803e-05" iyz="-1.5e-11" izz="1.35768e-05"/>
@@ -36,5 +36,5 @@
       <!-- Part camera_mount_base_link -->
       <visual>
-        <origin xyz="0 0 0" rpy="0 -0 0"/>
+        <origin xyz="0.000851685 0 -0.535218" rpy="0 -0 0"/>
         <geometry>
           <mesh filename="package://camera_mount_description/urdf/assets/camera_mount_base_link.stl"/>
@@ -45,5 +45,5 @@
       </visual>
       <collision>
-        <origin xyz="0 0 0" rpy="0 -0 0"/>
+        <origin xyz="0.000851685 0 -0.535218" rpy="0 -0 0"/>
         <geometry>
           <mesh filename="package://camera_mount_description/urdf/assets/camera_mount_base_link.stl"/>
@@ -52,5 +52,5 @@
       <!-- Part dc15_a01_case_f_dummy -->
       <visual>
-        <origin xyz="0.056648 0 0.550718" rpy="0 0 -1.5708"/>
+        <origin xyz="0.0574997 0 0.0155" rpy="0 0 -1.5708"/>
         <geometry>
           <mesh filename="package://camera_mount_description/urdf/assets/dc15_a01_case_f_dummy.stl"/>
@@ -61,5 +61,5 @@
       </visual>
       <collision>
-        <origin xyz="0.056648 0 0.550718" rpy="0 0 -1.5708"/>
+        <origin xyz="0.0574997 0 0.0155" rpy="0 0 -1.5708"/>
         <geometry>
           <mesh filename="package://camera_mount_description/urdf/assets/dc15_a01_case_f_dummy.stl"/>
@@ -68,5 +68,5 @@
       <!-- Part base_mount -->
       <visual>
-        <origin xyz="0 0 0" rpy="0 -0 -0"/>
+        <origin xyz="0.000851685 0 -0.535218" rpy="0 -0 -0"/>
         <geometry>
           <mesh filename="package://camera_mount_description/urdf/assets/base_mount.stl"/>
@@ -77,5 +77,5 @@
       </visual>
       <collision>
-        <origin xyz="0 0 0" rpy="0 -0 -0"/>
+        <origin xyz="0.000851685 0 -0.535218" rpy="0 -0 -0"/>
         <geometry>
           <mesh filename="package://camera_mount_description/urdf/assets/base_mount.stl"/>
@@ -160,5 +160,5 @@
     <!-- Joint from camera_mount_base_link to camera_mount_yaw_link -->
     <joint name="yaw" type="revolute">
-      <origin xyz="0.056648 0 0.557218" rpy="-3.14159 0 -1.5708"/>
+      <origin xyz="0.0574997 0 0.022" rpy="-3.14159 0 -1.5708"/>
       <parent link="camera_mount_base_link"/>
       <child link="camera_mount_yaw_link"/>
@@ -175,5 +175,5 @@
          (both d455 meshes, ours and realsense2_description's, share the same local
          origin convention, confirmed by comparing STL bounding boxes: identical
-         124x26x29mm dimensions, matching center offsets to sub-mm noise). -->
+         124x26x29mm dimensions, maching center offsets to sub-mm noise). -->
     <xacro:sensor_d455 parent="camera_mount_pitch_link" name="camera" use_nominal_extrinsics="true">
       <origin xyz="0.029198 -0.0145 0.0145" rpy="-1.570796 0 0"/>
